File: hellen-hyundai-pb-154.kicad_pcb (KiCad board)
At the start: 4 copper layers, 164 x 156 mm, 1 part

Commit message: GDI pinout
Parts:
- removed G2: DISCLAIMER, rusefi_lib:Off_Road_Disclaimer
- added F1: Fuse-Pad-Pad, hellen-one-common:PAD-1206-PAD, F.Cu at (184.2, -26.8)
- added F2: Fuse-Pad-Pad, hellen-one-common:PAD-1206-PAD, F.Cu at (402.0, 53.4)
- added F3: Fuse-Pad-Pad, hellen-one-common:PAD-1206-PAD, F.Cu at (402.0, 56.5)
- added F4: Fuse-Pad-Pad, hellen-one-common:PAD-1206-PAD, F.Cu at (178.7, -26.8)
- added F5: Fuse-Pad-Pad, hellen-one-common:PAD-1206-PAD, F.Cu at (402.0, 62.7)
- added J1: 6473423-1, kicad6-libraries:6473423-1, F.Cu at (238.5, -4.90)
- added P1: 284617-1, kicad6-libraries:TE_284617-1, F.Cu at (119.7, -33.5)
- added P2: Pad, hellen-one-common:PAD-TH, F.Cu at (399.9, 66.2)
- added P3: Pad, hellen-one-common:PAD-TH, F.Cu at (399.9, 69.9)
- added P4: Pad, hellen-one-common:PAD-TH, F.Cu at (399.9, 73.7)
- added P5: Pad, hellen-one-common:PAD-TH, F.Cu at (399.9, 77.5)
- added R1: Jumper-Pad-Pad, hellen-one-common:PAD-0805-PAD, F.Cu at (368.0, 50.1)
- added R10: Jumper-Pad-Pad, hellen-one-common:PAD-0805-PAD, F.Cu at (368.0, 75.8)
- added R11: Jumper-Pad-Pad, hellen-one-common:PAD-0805-PAD, F.Cu at (368.0, 78.6)
- added R12: Jumper-Pad-Pad, hellen-one-common:PAD-0805-PAD, F.Cu at (374.7, 50.1)
- added R13: Jumper-Pad-Pad, hellen-one-common:PAD-0805-PAD, F.Cu at (374.7, 52.9)
- added R14: Jumper-Pad-Pad, hellen-one-common:PAD-0805-PAD, F.Cu at (374.7, 55.8)
- added R15: Jumper-Pad-Pad, hellen-one-common:PAD-0805-PAD, F.Cu at (374.7, 58.6)
- added R16: Jumper-Pad-Pad, hellen-one-common:PAD-0805-PAD, F.Cu at (230.0, -30.7)
- added R17: Jumper-Pad-Pad, hellen-one-common:PAD-0805-PAD, F.Cu at (374.7, 64.3)
- added R18: Jumper-Pad-Pad, hellen-one-common:PAD-0805-PAD, F.Cu at (374.7, 67.2)
- added R19: Jumper-Pad-Pad, hellen-one-common:PAD-0805-PAD, F.Cu at (374.7, 70.1)
- added R2: Jumper-Pad-Pad, hellen-one-common:PAD-0805-PAD, F.Cu at (368.0, 52.9)
- added R20: Jumper-Pad-Pad, hellen-one-common:PAD-0805-PAD, F.Cu at (374.7, 72.9)
- added R21: Jumper-Pad-Pad, hellen-one-common:PAD-0805-PAD, F.Cu at (374.7, 75.8)
- added R22: Jumper-Pad-Pad, hellen-one-common:PAD-0805-PAD, F.Cu at (374.7, 78.6)
- added R23: Jumper-Pad-Pad, hellen-one-common:PAD-0805-PAD, F.Cu at (381.4, 50.1)
- added R24: Jumper-Pad-Pad, hellen-one-common:PAD-0805-PAD, F.Cu at (381.4, 52.9)
- added R25: Jumper-Pad-Pad, hellen-one-common:PAD-0805-PAD, F.Cu at (381.4, 55.8)
- added R26: Jumper-Pad-Pad, hellen-one-common:PAD-0805-PAD, F.Cu at (381.4, 58.6)
- added R27: Jumper-Pad-Pad, hellen-one-common:PAD-0805-PAD, F.Cu at (381.4, 61.5)
- added R28: Jumper-Pad-Pad, hellen-one-common:PAD-0805-PAD, F.Cu at (381.4, 64.3)
- added R29: Jumper-Pad-Pad, hellen-one-common:PAD-0805-PAD, F.Cu at (381.4, 67.2)
- added R3: Jumper-Pad-Pad, hellen-one-common:PAD-0805-PAD, F.Cu at (368.0, 55.8)
- added R30: Jumper-Pad-Pad, hellen-one-common:PAD-0805-PAD, F.Cu at (381.4, 70.1)
- added R31: Jumper-Pad-Pad, hellen-one-common:PAD-0805-PAD, F.Cu at (381.4, 72.9)
- added R32: Jumper-Pad-Pad, hellen-one-common:PAD-0805-PAD, F.Cu at (381.4, 75.8)
- added R33: Jumper-Pad-Pad, hellen-one-common:PAD-0805-PAD, F.Cu at (381.4, 78.6)
- added R34: Jumper-Pad-Pad, hellen-one-common:PAD-0805-PAD, F.Cu at (388.0, 50.1)
- added R35: Jumper-Pad-Pad, hellen-one-common:PAD-0805-PAD, F.Cu at (388.0, 52.9)
- added R36: Jumper-Pad-Pad, hellen-one-common:PAD-0805-PAD, F.Cu at (388.0, 55.8)
- added R37: Jumper-Pad-Pad, hellen-one-common:PAD-0805-PAD, F.Cu at (388.0, 58.6)
- added R38: Jumper-Pad-Pad, hellen-one-common:PAD-0805-PAD, F.Cu at (388.0, 61.5)
- added R39: Jumper-Pad-Pad, hellen-one-common:PAD-0805-PAD, F.Cu at (388.0, 64.3)
- added R4: Jumper-Pad-Pad, hellen-one-common:PAD-0805-PAD, F.Cu at (368.0, 58.6)
- added R40: Jumper-Pad-Pad, hellen-one-common:PAD-0805-PAD, F.Cu at (388.0, 67.2)
- added R41: Jumper-Pad-Pad, hellen-one-common:PAD-0805-PAD, F.Cu at (388.0, 70.1)
- added R42: Jumper-Pad-Pad, hellen-one-common:PAD-0805-PAD, F.Cu at (388.0, 72.9)
- added R43: Jumper-Pad-Pad, hellen-one-common:PAD-0805-PAD, F.Cu at (388.0, 75.8)
- added R44: Jumper-Pad-Pad, hellen-one-common:PAD-0805-PAD, F.Cu at (388.0, 78.6)
- added R45: Jumper-Pad-Pad, hellen-one-common:PAD-0805-PAD, F.Cu at (394.7, 50.1)
- added R46: Jumper-Pad-Pad, hellen-one-common:PAD-0805-PAD, F.Cu at (394.7, 52.9)
- added R47: Jumper-Pad-Pad, hellen-one-common:PAD-0805-PAD, F.Cu at (394.7, 55.8)
- added R48: Jumper-Pad-Pad, hellen-one-common:PAD-0805-PAD, F.Cu at (394.7, 58.6)
- added R49: Jumper-Pad-Pad, hellen-one-common:PAD-0805-PAD, F.Cu at (394.7, 61.5)
- added R5: Jumper-Pad-Pad, hellen-one-common:PAD-0805-PAD, F.Cu at (368.0, 61.5)
- added R50: Jumper-Pad-Pad, hellen-one-common:PAD-0805-PAD, F.Cu at (394.7, 64.3)
- added R51: Jumper-Pad-Pad, hellen-one-common:PAD-0805-PAD, F.Cu at (394.7, 67.2)
- added R52: Jumper-Pad-Pad, hellen-one-common:PAD-0805-PAD, F.Cu at (394.7, 70.1)
- added R53: Jumper-Pad-Pad, hellen-one-common:PAD-0805-PAD, F.Cu at (394.7, 72.9)
- added R54: Jumper-Pad-Pad, hellen-one-common:PAD-0805-PAD, F.Cu at (394.7, 75.8)
- added R55: Jumper-Pad-Pad, hellen-one-common:PAD-0805-PAD, F.Cu at (394.7, 78.6)
- added R6: Jumper-Pad-Pad, hellen-one-common:PAD-0805-PAD, F.Cu at (368.0, 64.3)
- added R7: Jumper-Pad-Pad, hellen-one-common:PAD-0805-PAD, F.Cu at (368.0, 67.2)
- added R8: Jumper-Pad-Pad, hellen-one-common:PAD-0805-PAD, F.Cu at (368.0, 70.1)
- added R9: Jumper-Pad-Pad, hellen-one-common:PAD-0805-PAD, F.Cu at (227.4, -30.8)
Routing:
- net /OUT_INJ2n: track 0.00 -> 60.9 mm
- net /OUT_INJ4p: track 0.00 -> 50.4 mm
- net /OUT_INJ3n: track 0.00 -> 33.1 mm
- net /OUT_INJ3p: track 0.00 -> 32.6 mm
- net /OUT_INJ1p: track 0.00 -> 31.1 mm
- net /OUT_INJ2p: track 0.00 -> 29.7 mm
- net /OUT_INJ4n: track 0.00 -> 17.7 mm
- net /OUT_INJ1n: track 0.00 -> 17.4 mm
- net /OUT_HS_FUEL_VALVE: track 0.00 -> 14.6 mm
- net /OUT_LS_FUEL_VALVE: track 0.00 -> 9.60 mm
- net Net-(P1-Pad49): track 0.00 -> 4.73 mm
