File: hellen-hyundai-pb-154.kicad_sch (KiCad schematic)
At the start: 4 parts, among them P1 284617-1, P2 Pad

Commit message: Pinout
Parts:
- added F2, F3, F4, F5: Fuse-Pad-Pad, hellen-one-common:PAD-1206-PAD, symbol hellen-one-common:Fuse-Pad-Pad
- added P3, P4, P5: Pad, hellen-one-common:PAD-TH, symbol hellen-one-common:Pad
- added R10, R11, R12, R13, R14, R15, R16, R17, R18, R19, R2, R20, R21, R22, R23, R24, R25, R26, R27, R28, R29, R3, R30, R31, R32, R33, R34, R35, R36, R37, R38, R39, R4, R40, R41, R42, R43, R44, R45, R46, R47, R48, R49, R5, R50, R51, R52, R53, R54, R55, R6, R7, R8, R9: Jumper-Pad-Pad, hellen-one-common:PAD-0805-PAD, symbol hellen-one-common:Jumper-Pad-Pad
Connections:
- net +12V_PERM: now also F2.2, F3.2
- net +12V_RAW: now also F1.2, F4.2
- net +5VP: now also P1.100 (40), P1.101 (41), P1.102 (42), P1.78 (18), P1.79 (19), P1.80 (20), P1.99 (39)
- net GND: now also P1.61 (1), P1.62 (2), P1.63 (3)
- net at F1.1: now also P1.64 (4)
- net at P2.1 (Pin_1): now also P1.90 (30)
- net OUT_INJ3p: now reaches P1.1
- net at P1.15: now also R2.2
- net OUT_INJ2p: now reaches P1.16
- net OUT_INJ1p: now reaches P1.17
- net OUT_INJ3n: now reaches P1.18
- net OUT_INJ4p: now reaches P1.2
- net at P1.20: now also R3.2
- net at P1.23: now also R4.2
- net GNDA: now reaches P1.24
- net GNDA: now also P1.115 (55), P1.124 (64), P1.136 (76), P1.137 (77), P1.138 (78), P1.146 (86), P1.38, P1.68 (8), P1.70 (10), P1.73 (13), P1.92 (32), P1.93 (33), P1.95 (35)
- net at P1.27: now also R5.2
- net at P1.29: now also R6.2
- net OUT_INJ2n: now reaches P1.3
- net at P1.31: now also R7.2
- net at P1.32: now also R8.2
- net OUT_INJ1n: now reaches P1.33
- net at P1.34: now also R9.2
- net at P1.35: now also R10.2
- net at P1.37: now also R11.2
- net at P1.40: now also R12.2
- net at P1.45: now also R13.2
- net at P1.46: now also R14.2
- net at P1.47: now also R15.2
- net OUT_INJ4n: now reaches P1.48
- net at P1.49: now also R16.2
- net at P1.5: now also R1.2
- net at P1.50: now also R17.2
- net at P1.53: now also R18.2
- net at P1.55: now also R19.2
- net at P1.57: now also R22.2
- net at P1.58: now also R21.2
- net at P1.59: now also R20.2
- net at P1.103 (43): now also R31.2
- net at P1.104 (44): now also R32.2
- net at P1.105 (45): now also R33.2
- net at P1.106 (46): now also R34.2
- net at P1.112 (52): now also R35.2
- net at P1.113 (53): now also R36.2
- net at P1.117 (57): now also R37.2
- net at P1.118 (58): now also R38.2
- net at P1.120 (60): now also R39.2
- net at P1.121 (61): now also R40.2
- net at P1.122 (62): now also P3.1 (Pin_1)
- net at P1.123 (63): now also R41.2
- net at P1.125 (65): now also R42.2
- net at P1.127 (67): now also R43.2
- net at P1.132 (72): now also R44.2
- net at P1.134 (74): now also R45.2
- net at P1.135 (75): now also R46.2
- net at P1.139 (79): now also R47.2
- net at P1.140 (80): now also R48.2
- net at P1.143 (83): now also P4.1 (Pin_1)
- net at P1.144 (84): now also P5.1 (Pin_1)
- net at P1.145 (85): now also R49.2
- net at P1.147 (87): now also R50.2
- net at P1.149 (89): now also R51.2
- net at P1.150 (90): now also R52.2
- net at P1.152 (92): now also R53.2
- net at P1.153 (93): now also R54.2
- net at P1.154 (94): now also R55.2
- net at P1.65 (5): now also F2.1
- net at P1.66 (6): now also F3.1
- net at P1.67 (7): now also F4.1
- net at P1.69 (9): now also R23.2
- net at P1.74 (14): now also R24.2
- net at P1.77 (17): now also R25.2
- net at P1.82 (22): now also R26.2
- net at P1.84 (24): now also R27.2
- net at P1.89 (29): now also F5.1
- net at P1.91 (31): now also R28.2
- net at P1.96 (36): now also R29.2
- net at P1.97 (37): now also R30.2
- net OUT_WBO_HTR: now reaches R1.1
- new net ALT_COM: R22.1
- new net CANH: R49.1
- new net CANL: R41.1
- new net IN_AC_PRESSURE: R33.1
- new net IN_AC_PRESSURE_SWITCH: R32.1
- new net IN_AC_SWITCH: R31.1
- new net IN_AMBIENT_TEMP: R30.1
- new net IN_BOOST_PRESSURE: R37.1
- new net IN_CLT: R4.1
- new net IN_EXHAUST_CAM: R42.1
- new net IN_FUEL_LEVEL: R25.1
- new net IN_HIGH_FUEL_PRESSURE: R38.1
- new net IN_HS_BRAKE: R18.1
- new net IN_HS_HOT_BRAKE: R12.1
- new net IN_HS_START_REQUEST: R39.1
- new net IN_HS_WIPER: R26.1
- new net IN_IAT: R47.1
- new net IN_INTAKE_CAM: R50.1
- new net IN_KNOCK: R11.1
- new net IN_LIN: R40.1
- new net IN_LS_CLUTCH: R19.1
- new net IN_MAP: R48.1
- new net IN_PPS1: R23.1
- new net IN_PPS2: R28.1
- new net IN_TPS1: R24.1
- new net IN_TPS2: R29.1
- new net IN_VIGN: F5.2
- new net IN_VR_CRANKn: R43.1
- new net IN_VR_CRANKp: R51.1
- new net IN_VSS: R34.1
- new net OUT_ALT_PWM: R27.1
- new net OUT_ETBn: R10.1
- new net OUT_ETBp: R17.1
- new net OUT_FAN_PWM: R20.1
- new net OUT_HS_FUEL_VALVE: R9.1
- new net OUT_IGN1: R8.1
- new net OUT_IGN2: R15.1
- new net OUT_IGN3: R7.1
- new net OUT_IGN4: R14.1
- new net OUT_LS_AC_REL: R6.1
- new net OUT_LS_EXHAUST_VVT: R2.1
- new net OUT_LS_FUEL_PUMP_REL: R5.1
- new net OUT_LS_FUEL_PUMP_REL2: R52.1
- new net OUT_LS_FUEL_VALVE: R16.1
- new net OUT_LS_INTAKE_VVT: R13.1
- new net OUT_LS_MAIN_REL: R54.1
- new net OUT_LS_PURGE_VALVE: R44.1
- new net OUT_LS_STARTER_REL: R55.1
- new net OUT_O2_HTR: R3.1
- new net OUT_TACH: R21.1
- new net OUT_WASTEGATE: R53.1
- new net WBO_NERNST_VOLTAGE: R45.1
- new net WBO_PUMPING_CURRENT: R36.1
- new net WBO_TRIM: R46.1
- new net WBO_VIRTUAL_GND: R35.1
- no-connect marks 0 -> 58
Other:
- note added: "?"
- note added: "Downstream O2 Signal"
- note added: "IMMO"
- note added: "PU"
- moved on the sheet: F1, P1A, P1B, R1

Commit message: GDI pinout
Parts:
- added J1: 6473423-1, kicad6-libraries:6473423-1, symbol TE_6473423-1:6473423-1
Connections:
- net +12V_RAW: now also J1.14 (14D), J1.20 (20D)
- net CANH: now also J1.12 (12D)
- net CANL: now also J1.11 (11D)
- net GND: now also J1.10 (10D), J1.9 (9D)
- net OUT_HS_FUEL_VALVE: now also J1.8 (8D)
- net OUT_INJ1n: now also J1.3 (3D)
- net OUT_INJ1p: now also J1.5 (5D)
- net OUT_INJ2n: now also J1.19 (19D)
- net OUT_INJ2p: now also J1.6 (6D)
- net OUT_INJ3n: now also J1.4 (4D)
- net OUT_INJ3p: now also J1.7 (7D)
- net OUT_INJ4n: now also J1.2 (2D)
- net OUT_INJ4p: now also J1.13 (13D)
- net OUT_LS_FUEL_VALVE: now also J1.1 (1D)
- new net GDI_INJ1: J1.21 (21D)
- new net GDI_INJ2: J1.22 (22D)
- new net GDI_INJ3: J1.23 (23D)
- new net GDI_INJ4: J1.24 (24D)
- new net GDI_PUMP1: J1.25 (25D)
- new net GDI_PUMP2: J1.26 (26D)

Commit message: Upd SCH
Parts:
- removed R3: Jumper-Pad-Pad, hellen-one-common:PAD-0805-PAD, symbol hellen-one-common:Jumper-Pad-Pad
- added BT1: BATTERY_CR2032, Battery:BatteryHolder_Keystone_1060_1x2032, symbol art-electro-power:BATTERY_CR2032
- added C1: 100n, hellen-one-common:C0603, symbol hellen-one-common:Cap
- added C2: 10u, hellen-one-common:C0603, symbol hellen-one-common:Cap
- added D1: 1N4148WS, hellen-one-common:SOD-323, symbol hellen-one-common:1N4148WS
- added J2: Conn_01x06, Connector_PinHeader_2.54mm:PinHeader_1x06_P2.54mm_Vertical, symbol Connector_Generic:Conn_01x06
- added J3: USB_B, Connector_USB:USB_B_OST_USB-B1HSxx_Horizontal, symbol Connector:USB_B
- added J4: Conn_01x05_Male, Connector_JST:JST_EH_B5B-EH-A_1x05_P2.50mm_Vertical, symbol Connector:Conn_01x05_Pin
- added J5: AudioJack3_SwitchTR, hellen-one-common:Jack_3.5mm_PJ-3250-5A, symbol Connector:AudioJack3_SwitchTR
- added M1: Module-wbo-0.5, hellen-one-wbo-0.5:wbo, symbol hellen-one-wbo-0.5:Module-wbo-0.5
- added M2: Module-mega-mcu144-0.4, hellen-one-mega-mcu144-0.4:mega-mcu144, symbol mega-mcu144-0.4:Module-mega-mcu144-0.4
- added M3: Module-stlink-0.1, hellen-one-stlink-0.1:stlink, symbol hellen-one-stlink-0.1:Module-stlink-0.1
- added M4: Module-power_12and5V-0.1, hellen-one-power_12and5V-0.1:power_12and5V, symbol power_12and5V-0.1:Module-power_12and5V-0.1
- added M5: Module-output-0.3, hellen-one-output-0.3:output, symbol hellen-one-output-0.3:Module-output-0.3
- added M6: Module-knock-0.2, hellen-one-knock-0.2:knock, symbol hellen-one-knock-0.2:Module-knock-0.2
- added P6, P7: Pad, hellen-one-common:PAD-TH, symbol hellen-one-common:Pad
- added U1: MCP6002-xSN, Package_SO:SOIC-8_3.9x4.9mm_P1.27mm, symbol Amplifier_Operational:MCP6002-xSN
Connections:
- net +12V_PERM: now also M4.V1 (V12_PERM)
- net +12V_RAW: now also M4.V3 (V12_RAW), M5.S11 (V12_RAW)
- net +5VP: now also M4.V4 (5VP)
- net CANH: now also M2.W12 (CANH)
- net CANL: now also M2.W13 (CANL)
- net GND: now also BT1.2 (-), C1.1, J2.3 (Pin_3), J3.4 (GND), J3.5 (Shield), J4.4 (Pin_4), J4.5 (Pin_5), J5.S, M1.E6 (LSU_H-), M1.G (GND), M2.G (GND), M3.G (GND), M4.S1 (GND), M5.G (GND), M5.S3 (GND), M6.E2 (GND), U1.4 (V-), U1.5 (+)
- net GNDA: now also M2.E39 (GNDA), M2.W1 (GNDA)
- net IN_KNOCK: now also M6.W1 (IN_KNOCK)
- net IN_VIGN: now also M4.V2 (IN_VIGN)
- net OUT_WBO_HTR: no longer R1.1
- net WBO_NERNST_VOLTAGE: no longer R45.1
- net WBO_TRIM: no longer R46.1
- net WBO_VIRTUAL_GND: no longer R35.1
- net at P1.20: now also P6.1 (Pin_1)
- net WBO_PUMPING_CURRENT renamed WBO_Ip
- net WBO_Ip: now also M1.E3 (LSU_Ip)
- new net: C2.2, U1.1, U1.2 (-)
- new net: BT1.1 (+), D1.2 (A)
- new net: U1.6 (-), U1.7
- new net: M2.N1 (USBID), P7.1 (Pin_1)
- new net: J2.1 (Pin_1), M1.W8 (V33_OUT)
- new net: J2.2 (Pin_2), M1.W7 (SWCLK)
- new net: J2.4 (Pin_4), M1.W6 (SWDIO)
- new net: J2.5 (Pin_5), M1.W5 (nReset)
- new net: M1.J1 (SEL1), M1.J_GND1 (PULL_DOWN1)
- new net: C2.1, J5.T
- new net: M2.N6 (SWO), M3.N3 (SWO)
- new net: M2.N7 (SWDIO), M3.N4 (SWDIO)
- new net: M2.N8 (SWCLK), M3.N5 (SWCLK)
- new net: M2.N9 (nReset), M3.N6 (nReset)
- new net +12V: M4.E2 (V12)
- new net +12V_PROT: M4.E5 (EN_5VP), M5.W5 (V12P)
- new net +3.3VA: M2.N28 (V33_SWITCHABLE)
- new net +3V3: M2.N22 (V33), M2.N32 (V33), M3.N2 (V33)
- new net +5V: C1.2, M2.N31 (VCC), M3.N1 (V5), M4.E4 (V5), M5.W14 (V5), U1.8 (V+)
- new net +5VA: M1.W1 (V5_IN), M2.E38 (V5A_SWITCHABLE), M2.W2 (V5A_SWITCHABLE), M6.E1 (V5A)
- new net CAN_H: M1.W4 (CANH)
- new net CAN_L: M1.W3 (CANL)
- new net KNOCK: M2.S23 (IN_KNOCK), M6.E3 (OUT_KNOCK), U1.3 (+)
- new net PG_5VP: M2.S1 (IN_D4), M4.E6 (PG_5VP)
- new net USB+: J3.3 (D+), J4.3 (Pin_3), M2.N3 (USBP)
- new net USB-: J3.2 (D-), J4.2 (Pin_2), M2.N2 (USBM)
- new net V33_REF: M1.W9 (VDDA), M2.W3 (V33_REF)
- new net VBAT: D1.1 (K), M2.N27 (VBAT), M4.E1 (VBAT)
- new net VBUS: J3.1 (VBUS), J4.1 (Pin_1), M2.N4 (VBUS)
- new net VIGN: M2.N26 (IN_VIGN), M4.E3 (VIGN)
- new net VREF2: M2.S5 (VREF2), M6.W2 (VREF)
- new net WBO_H-: M1.E5 (LSU_H+), R1.1
- new net WBO_R_Trim: M1.E4 (LSU_Rtrim), R46.1
- new net WBO_Vs: M1.E1 (LSU_Un), R45.1
- new net WBO_Vs/Ip: M1.E2 (LSU_Vm), R35.1
- no-connect marks 58 -> 71
Other:
- added sheet ETB (ETB.kicad_sch)
- note added: "Power"
- moved on the sheet: J1

Commit message: Upd SCH
Parts:
- removed C1: 100n, hellen-one-common:C0603, symbol hellen-one-common:Cap
- removed C2: 10u, hellen-one-common:C0603, symbol hellen-one-common:Cap
- removed J5: AudioJack3_SwitchTR, hellen-one-common:Jack_3.5mm_PJ-3250-5A, symbol Connector:AudioJack3_SwitchTR
- removed M6: Module-knock-0.2, hellen-one-knock-0.2:knock, symbol hellen-one-knock-0.2:Module-knock-0.2
- removed R14, R15, R7, R8: Jumper-Pad-Pad, hellen-one-common:PAD-0805-PAD, symbol hellen-one-common:Jumper-Pad-Pad
- removed U1: MCP6002-xSN, Package_SO:SOIC-8_3.9x4.9mm_P1.27mm, symbol Amplifier_Operational:MCP6002-xSN
- added F6, F7, F8, F9: Fuse-16A, hellen-one-common:36911600000, symbol hellen-one-common:Fuse-Pad-Pad
- added M7: Module-vr-discrete-0.4, hellen-one-vr-discrete-0.4:vr-discrete, symbol vr-discrete-0.4:Module-vr-discrete-0.4
- added M8: Module-lin-0.1, hellen-one-lin-0.1:lin, symbol hellen-one-lin-0.1:Module-lin-0.1
- added R60: 4.7k, hellen-one-common:R0603, symbol hellen-one-common:Res
Connections:
- net OUT_LS_FUEL_PUMP_REL2 is gone; now on net OUT_LS_FUEL_PUMP_REL: R52.1
- net +12V: now also M8.N1 (12V), M8.V1 (12V)
- net +3V3: now also R60.1
- net +5VA: now also M7.E4 (V5_IN), M8.V3 (5V)
- net GDI_INJ1: now also M2.E19 (OUT_INJ1)
- net GDI_INJ2: now also M2.E18 (OUT_INJ2)
- net GDI_INJ3: now also M2.E29 (OUT_INJ3)
- net GDI_INJ4: now also M2.E30 (OUT_INJ4)
- net GDI_PUMP1: now also M2.E31 (OUT_INJ5)
- net GDI_PUMP2: now also M2.E32 (OUT_INJ6)
- net GND: now also M7.G (GND), M8.E1 (GND), M8.S1 (GND)
- net IN_AC_PRESSURE: now also M2.S11 (IN_AUX3)
- net IN_AC_PRESSURE_SWITCH: now also M2.S2 (IN_D3)
- net IN_AC_SWITCH: now also M2.S3 (IN_D2)
- net IN_AMBIENT_TEMP: now also M2.S12 (IN_AUX2)
- net IN_BOOST_PRESSURE: now also M2.S16 (IN_O2S)
- net IN_CLT: now also M2.S28 (IN_CLT)
- net IN_EXHAUST_CAM: now also M2.S14 (IN_RES2)
- net IN_FUEL_LEVEL: now also M2.S13 (IN_AUX1)
- net IN_HIGH_FUEL_PRESSURE: now also M2.S15 (IN_O2S2)
- net IN_HS_BRAKE: now also M2.S8 (IN_SENS2)
- net IN_HS_HOT_BRAKE: now also M2.S9 (IN_SENS1)
- net IN_HS_START_REQUEST: now also M2.S4 (IN_D1)
- net IN_HS_WIPER: now also M2.S6 (IN_SENS4)
- net IN_IAT: now also M2.S26 (IN_IAT)
- net IN_INTAKE_CAM: now also M2.S17 (IN_RES1)
- net IN_LIN: now also M8.V4 (LIN)
- net IN_LS_CLUTCH: now also M2.S7 (IN_SENS3)
- net IN_MAP: now also M2.S21 (IN_MAP1)
- net IN_PPS1: now also M2.S31 (IN_PPS)
- net IN_PPS2: now also M2.S33 (IN_PPS2)
- net IN_TPS1: now also M2.S30 (IN_TPS)
- net IN_TPS2: now also M2.S32 (IN_TPS2)
- net IN_VR_CRANKn: now also M7.W1 (VR-)
- net IN_VR_CRANKp: now also M7.W2 (VR+)
- net IN_VSS: now also M2.S25 (IN_VSS)
- net OUT_IGN1: now also F7.2
- net OUT_IGN2: now also F9.2
- net OUT_IGN3: now also F6.2
- net OUT_IGN4: now also F8.2
- net OUT_LS_AC_REL: now also M5.W1 (OUT_LOW2)
- net OUT_LS_FUEL_PUMP_REL: now also M5.S8 (OUT_LOW1)
- net OUT_LS_MAIN_REL: now also M5.W13 (OUT_LOW5_MAIN)
- net OUT_LS_STARTER_REL: now also M5.W3 (OUT_LOW6_DIODE)
- net at P1.46: now also F8.1
- net at M5.W21 (LOW1): now also M2.E8 (OUT_IO1)
- net at M5.W25 (LOW6_DIODE): now also M2.E9 (OUT_IO6)
- net at M5.W26 (LOW10): now also M2.E10 (OUT_IO10)
- net at M5.W27 (LOW9): now also M2.E11 (OUT_IO9)
- net at M5.W29 (LOW2): now also M2.E12 (OUT_IO2)
- net at M5.W34 (LOW4_DUAL): now also M2.E21 (OUT_IO4)
- net at M5.W35 (LOW11): now also M2.E24 (OUT_IO11)
- net at M5.W36 (LOW12): now also M2.E13 (OUT_IO12)
- net at M5.W37 (LOW8_HIGH2): now also M2.E22 (OUT_IO8)
- net at M5.W38 (LOW3_DUAL): now also M2.E6 (OUT_IO3)
- net at M5.W39 (LOW7_HIGH1): now also M2.E23 (OUT_IO7)
- net at M5.W40 (LOW5_MAIN): now also M2.E7 (OUT_IO5)
- net at P1.31: now also F6.1
- net at P1.32: now also F7.1
- net at P1.47: now also F9.1
- net ETB_DIS: now reaches M2.E16 (OUT_PWM3)
- net ETB_DIR: now reaches M2.E17 (OUT_PWM2)
- net ETB_PWM: now reaches M2.E27 (OUT_PWM1)
- net CRANK_THR: now reaches M2.E28 (OUT_PWM8)
- net CRANK_THR: now also M7.E1 (Thresh_IN)
- net at M2.N17 (UART2_TX): now also M8.V5 (UART_TX)
- net at M2.N18 (UART2_RX): now also M8.V2 (UART_RX), R60.2
- net CRANK_A: now reaches M2.S18 (IN_RES3)
- net CRANK_A: now also M7.E2 (OUT_A)
- net CRANK: now reaches M2.S22 (IN_CRANK)
- net CRANK: now also M7.E3 (OUT)
- net DUMB_COILS/IN2: now reaches M2.W10 (IGN2)
- net DUMB_COILS/IN1: now reaches M2.W11 (IGN1)
- net DUMB_COILS/IN4: now reaches M2.W8 (IGN4)
- net DUMB_COILS/IN3: now reaches M2.W9 (IGN3)
- net OUT_WASTEGATE renamed OUT_LS_WASTEGATE
- no-connect marks 71 -> 76
Other:
- added sheet DUMB_COILS (DUBM_COILS4.kicad_sch)
- added sheet KNOCK (KNOCK.kicad_sch)
- note added: "TODO: R slave?"
- moved on the sheet: J1, J2, M1, M5A, M5B, M5C
